File: Electrical/PCB/Control Board/Control Board.sch (KiCad schematic (older format))
At the start: 88 parts, among them J1 ED2627-ND, J10 6posheader, J11 S7038-ND, J12 ED2989-ND-USB, J13 ED1501-ND, J14 ED2989-ND-USB, J15 ED2580-ND, J16 ED2580-ND, J17 ED2744-ND, J18 ED2744-ND, J19 ED2744-ND, J2 ED2627-ND, J20 ED2744-ND, J21 ED2744-ND, J22 ED2744-ND, J23 ED2744-ND, J24 ED2744-ND, J25 ED2744-ND, J26 ED2744-ND, J3 ED2627-ND, J4 ED2627-ND, J5 ED2627-ND, J6 S9175-ND, J7 S9175-ND, J8 6posheader, J9 S7038-ND, M1 Mounting_Holes, T1 test_point, T10 test_point, T11 test_point, T12 test_point, T13 test_point, T14 test_point, T15 test_point, T16 test_point, T17 test_point, T18 test_point, T19 test_point, T2 test_point, T20 test_point, T21 test_point, T3 test_point, T4 test_point, T5 test_point, T6 test_point, T7 test_point, T8 test_point, T9 test_point, U1 LM358-N, U2 LM358-N

Commit message: Adding board Rev-E of control board with updated silkscreen images, and Rev-D of arduino board also with silk screen fixes
Parts:
- added y1: rover_silkscreen, JPL Robotics:rover_image, symbol Control-Board-rescue:rover_silkscreen-Monolithic-Board-rescue
- J1, J2, J3, J4, J5: symbol Monolithic-Board-rescue:ED2627-ND-JPL_Robotics_Lib -> Control-Board-rescue:ED2627-ND-JPL_Robotics_Lib-Monolithic-Board-rescue
- J10, J8: symbol Monolithic-Board-rescue:6posheader-JPL_Robotics_Lib -> Control-Board-rescue:6posheader-JPL_Robotics_Lib-Monolithic-Board-rescue
- J11, J9: symbol Monolithic-Board-rescue:S7038-ND-JPL_Robotics_Lib -> Control-Board-rescue:S7038-ND-JPL_Robotics_Lib-Monolithic-Board-rescue
- J12, J14: symbol Monolithic-Board-rescue:ED2989-ND-USB-JPL_Robotics_Lib -> Control-Board-rescue:ED2989-ND-USB-JPL_Robotics_Lib-Monolithic-Board-rescue
- J13: symbol Monolithic-Board-rescue:ED1501-ND-JPL_Robotics_Lib -> Control-Board-rescue:ED1501-ND-JPL_Robotics_Lib-Monolithic-Board-rescue
- J15, J16: symbol Monolithic-Board-rescue:ED2580-ND-JPL_Robotics_Lib -> Control-Board-rescue:ED2580-ND-JPL_Robotics_Lib-Monolithic-Board-rescue
- J17, J18, J19, J20, J21, J22, J23, J24, J25, J26: symbol Monolithic-Board-rescue:ED2744-ND-JPL_Robotics_Lib -> Control-Board-rescue:ED2744-ND-JPL_Robotics_Lib-Monolithic-Board-rescue
- J6, J7: symbol Monolithic-Board-rescue:S9175-ND-JPL_Robotics_Lib -> Control-Board-rescue:S9175-ND-JPL_Robotics_Lib-Monolithic-Board-rescue
- M1: symbol Monolithic-Board-rescue:Mounting_Holes-JPL_Robotics_Lib -> Control-Board-rescue:Mounting_Holes-JPL_Robotics_Lib-Monolithic-Board-rescue
- MH1, MH2, MH3, MH4: symbol Monolithic-Board-rescue:#6THRU-HOLE-JPL_Robotics_Lib -> Control-Board-rescue:#6THRU-HOLE-JPL_Robotics_Lib-Monolithic-Board-rescue
- RC1, RC2, RC3, RC4, RC5: symbol Monolithic-Board-rescue:RoboClaw-JPL_Robotics_Lib -> Control-Board-rescue:RoboClaw-JPL_Robotics_Lib-Monolithic-Board-rescue
- T1, T10, T11, T12, T13, T14, T15, T16, T17, T18, T19, T2, T20, T21, T3, T4, T5, T6, T7, T8, T9: symbol Monolithic-Board-rescue:test_point-JPL_Robotics_Lib -> Control-Board-rescue:test_point-JPL_Robotics_Lib-Monolithic-Board-rescue
- U1, U2: symbol Monolithic-Board-rescue:LM358-N-JPL_Robotics_Lib -> Control-Board-rescue:LM358-N-JPL_Robotics_Lib-Monolithic-Board-rescue
