File: electrical/pcb/control_board/motor_board.sch (KiCad schematic (older format))
At the start: 101 parts, among them J1 ED2627-ND, J11 S7038-ND, J12 PEC10DAAN, J13 ED1501-ND, J14 ED2989-ND-USB, J15 ED2580-ND, J16 ED2580-ND, J17 Molex_172675-0613, J18 Molex_172675-0613, J19 Molex_172675-0613, J2 ED2627-ND, J20 Molex_172675-0613, J21 Molex_172675-0613, J22 Molex_172675-0613, J23 Molex_172675-0613, J24 Molex_172675-0613, J25 Molex_172675-0613, J26 Molex_172675-0613, J28 ED2580-ND, J29 ED2580-ND, J3 ED2627-ND, J30 ED2580-ND, J31 ED2580-ND, J33 ina260_Vin, J34 ina260_8pin, J4 ED2627-ND, J5 ED2627-ND, J9 S7038-ND, M1 Mounting_Holes, T1 test_point, T10 test_point, T11 test_point, T12 test_point, T13 test_point, T14 test_point, T15 test_point, T16 test_point, T17 test_point, T18 test_point, T19 test_point, T2 test_point, T20 test_point, T21 test_point, T3 test_point, T4 test_point, T5 test_point, T6 test_point, T7 test_point, T8 test_point, T9 test_point, U1 LM358-N, U2 LM358-N, y1 rover_silkscreen

Commit message: Adding xt60 connectors
Parts:
- removed J31: ED2580-ND, JPL Robotics:ED2580-ND, symbol JPL_Robotics_Lib:ED2580-ND
- J13: value ED1501-ND -> XT60-F; footprint JPL Robotics:ED1501-ND -> (none); symbol JPL_Robotics_Lib:ED1501-ND -> JPL_Robotics_Lib:XT60-F
- J15, J16, J28, J29, J30: value ED2580-ND -> XT60-F; footprint JPL Robotics:ED2580-ND -> (none); symbol JPL_Robotics_Lib:ED2580-ND -> JPL_Robotics_Lib:XT60-F
Connections:
- wire segments 400 -> 399
Other:
- note removed: "Adafruit INA260 v+/-"
Changed lines of the file:
@@
 RC5EN2A
 $Comp
-L JPL_Robotics_Lib:ED2580-ND J?
+L JPL_Robotics_Lib:XT60-F J?
 U 1 1 60B75381
 P 1700 6000
@@
 AR Path="/60A51BAC/60B75381" Ref="J15"  Part="1"
 F 0 "J15" V 1600 6150 30  0000 R CNN
-F 1 "ED2580-ND" V 1550 6200 30  0001 R CNN
-F 2 "JPL Robotics:ED2580-ND" H 1700 6200 30  0001 C CNN
+F 1 "XT60-F" V 1550 6200 30  0001 R CNN
+F 2 "" H 1700 6200 30  0001 C CNN
 F 3 "" H 1700 6200 30  0001 C CNN
 	1    1700 6000
@@
 	1400 8800 1300 8800
 $Comp
-L JPL_Robotics_Lib:ED1501-ND J?
+L JPL_Robotics_Lib:XT60-F J?
 U 1 1 60B75504
-P 2050 8800
+P 2100 8800
 AR Path="/60B75504" Ref="J?"  Part="1"
 AR Path="/60A51BAC/60B75504" Ref="J13"  Part="1"
-F 0 "J13" H 2156 9115 50  0000 C CNN
-F 1 "ED1501-ND" H 2156 9024 50  0000 C CNN
-F 2 "JPL Robotics:ED1501-ND" H 2050 8800 50  0001 C CNN
-F 3 "" H 2050 8800 50  0001 C CNN
-	1    2050 8800
+F 0 "J13" H 2050 9050 50  0000 C CNN
+F 1 "XT60-F" H 2206 9024 50  0001 C CNN
+F 2 "" H 2100 8800 50  0001 C CNN
+F 3 "" H 2100 8800 50  0001 C CNN
+	1    2100 8800
 	1    0    0    -1
 $EndComp
@@
 +BATT
 $Comp
-L JPL_Robotics_Lib:ED2580-ND J?
+L JPL_Robotics_Lib:XT60-F J?
 U 1 1 60B75520
 P 4500 7750
@@
 AR Path="/60A51BAC/60B75520" Ref="J28"  Part="1"
 F 0 "J28" V 4400 7900 30  0000 R CNN
-F 1 "ED2580-ND" V 4350 7950 30  0001 R CNN
-F 2 "JPL Robotics:ED2580-ND" H 4500 7950 30  0001 C CNN
+F 1 "XT60-F" V 4350 7950 30  0001 R CNN
+F 2 "" H 4500 7950 30  0001 C CNN
 F 3 "" H 4500 7950 30  0001 C CNN
 	1    4500 7750
@@
 	4350 6900 4350 7650
 $Comp
-L JPL_Robotics_Lib:ED2580-ND J?
+L JPL_Robotics_Lib:XT60-F J?
 U 1 1 60B75529
 P 2350 6000
@@
 AR Path="/60A51BAC/60B75529" Ref="J29"  Part="1"
 F 0 "J29" V 2250 6150 30  0000 R CNN
-F 1 "ED2580-ND" V 2200 6200 30  0001 R CNN
-F 2 "JPL Robotics:ED2580-ND" H 2350 6200 30  0001 C CNN
+F 1 "XT60-F" V 2200 6200 30  0001 R CNN
+F 2 "" H 2350 6200 30  0001 C CNN
 F 3 "" H 2350 6200 30  0001 C CNN
 	1    2350 6000
@@
 $EndComp
 $Comp
-L JPL_Robotics_Lib:ED2580-ND J?
+L JPL_Robotics_Lib:XT60-F J?
 U 1 1 60B7552F
 P 3800 6000
@@
 AR Path="/60A51BAC/60B7552F" Ref="J30"  Part="1"
 F 0 "J30" V 3700 6150 30  0000 R CNN
-F 1 "ED2580-ND" V 3650 6200 30  0001 R CNN
-F 2 "JPL Robotics:ED2580-ND" H 3800 6200 30  0001 C CNN
+F 1 "XT60-F" V 3650 6200 30  0001 R CNN
+F 2 "" H 3800 6200 30  0001 C CNN
 F 3 "" H 3800 6200 30  0001 C CNN
 	1    3800 6000
@@
 Switch
 $Comp
-L JPL_Robotics_Lib:ED2580-ND J?
+L JPL_Robotics_Lib:XT60-F J?
 U 1 1 60B75546
 P 3100 6000
@@
 AR Path="/60A51BAC/60B75546" Ref="J16"  Part="1"
 F 0 "J16" V 3000 6150 30  0000 R CNN
-F 1 "ED2580-ND" V 2950 6200 30  0001 R CNN
-F 2 "JPL Robotics:ED2580-ND" H 3100 6200 30  0001 C CNN
+F 1 "XT60-F" V 2950 6200 30  0001 R CNN
+F 2 "" H 3100 6200 30  0001 C CNN
 F 3 "" H 3100 6200 30  0001 C CNN
 	1    3100 6000
@@
 Text Label 2850 7450 0    30   ~ 0
 SWIN
-$Comp
-L JPL_Robotics_Lib:ED2580-ND J?
-U 1 1 60B75561
-P 2200 6750
-AR Path="/60B75561" Ref="J?"  Part="1"
-AR Path="/60A51BAC/60B75561" Ref="J31"  Part="1"
-F 0 "J31" V 2100 6900 30  0000 R CNN
-F 1 "ED2580-ND" V 2050 6950 30  0001 R CNN
-F 2 "JPL Robotics:ED2580-ND" H 2200 6950 30  0001 C CNN
-F 3 "" H 2200 6950 30  0001 C CNN
-	1    2200 6750
-	0    -1   -1   0
-$EndComp
-Wire Wire Line
-	1600 6600 2100 6600
-Wire Wire Line
-	2150 6600 2750 6600
-Text Notes 1400 6950 0    50   ~ 0
-Adafruit INA260 v+/-
 Text Notes 10300 6100 0    39   ~ 0
 note: opamps are used to \nbuffer raw encoder signals
@@
 	1    0    0    -1
 $EndComp
+Wire Wire Line
+	1600 6600 2750 6600
 $EndSCHEMATC
