File: electrical/pcb/control_board/Brain_Board.kicad_sch (KiCad schematic)
At the start: 52 parts, among them J22 S9175-ND_rpi_breakout, J23 S9175-ND_rpi_breakout, J24 6posheader, J25 SSW-104-01-F-T, J26 WM6548-ND, J27 PPTC021LFBN-RC, J28 PPTC021LFBN-RC, J29 PPTC021LFBN-RC, J30 PEC08SAAN, M1 Mounting_Holes, Q2 2N3906, Q3 2N3906, Q4 2N3906, Q5 2N3906, Q6 2N3906, SW1 CT206124-ND, T13 test_point, T14 test_point, T15 test_point, U6 DC7G3HWA, y2 rover_silkscreen

Commit message: Set U5/U6 to DC10CGKWA in board files and A37's Digi-Key cell
Parts:
- U6: value DC7G3HWA -> DC10CGKWA
Changed lines of the file:
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@@
 			)
 		)
-		(property "Value" "DC7G3HWA"
+		(property "Value" "DC10CGKWA"
 			(at 137.16 145.4404 0)
 			(show_name no)
