File: electrical/pcb/control_board/Motor_Board.kicad_sch (KiCad schematic)
At the start: 98 parts, among them J1 XT30-M, J10 Molex_172675-0613, J11 Molex_172675-0613, J12 TSW-104-07-F-T, J13 Molex_172675-0613, J14 Molex_172675-0613, J15 TSW-104-07-F-T, J16 277-11404-ND, J17 277-11404-ND, J18 277-11404-ND, J19 TSW-104-07-F-T, J2 ED2580-ND, J20 PEC08SAAN, J21 PPTC102LFBN-RC, J3 XT30-F, J4 XT30-F, J5 XT30-M, J6 ED2580-ND, J7 TSW-104-07-F-T, J8 Molex_172675-0613, J9 Molex_172675-0613, Q1 2N3906, T1 test_point, T10 test_point, T11 test_point, T12 test_point, T2 test_point, T3 test_point, T4 test_point, T5 test_point, T6 test_point, T7 test_point, T8 test_point, T9 test_point, U1 INA260, U2 PCA9685, U3 D24V22Fx, U4 D24V150Fx, U5 DC7G3HWA, U7 MIC2937A-3.3WT, y1 rover_silkscreen

Commit message: Set U5/U6 to DC10CGKWA in board files and A37's Digi-Key cell
Parts:
- U5: value DC7G3HWA -> DC10CGKWA
Changed lines of the file:
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@@
 			)
 		)
-		(property "Value" "DC7G3HWA"
+		(property "Value" "DC10CGKWA"
 			(at 372.11 119.38 0)
 			(show_name no)
