File: electrical/pcb/arduino_uno_shield/Arduino_uno_shield.sch (KiCad schematic (older format))
At the start: 16 parts, among them J1 ED10523-ND, J2 6posheader, J3 6posheader, J4 6posheader, J5 6posheader, J6 ED2580-ND, y1 rover_silkscreen

Commit message: Rename all the arduino "sheild" files to "shield"
Parts:
- A1: footprint JPL Robotics:Arduino Uno Sheild -> JPL Robotics:Arduino Uno Shield; symbol Arduino_uno_sheild-rescue:Arduino_UNO_R3-JPL_Robotics_Lib -> Arduino_uno_shield-rescue:Arduino_UNO_R3-JPL_Robotics_Lib
- J1: symbol Arduino_uno_sheild-rescue:ED10523-ND-JPL_Robotics_Lib -> Arduino_uno_shield-rescue:ED10523-ND-JPL_Robotics_Lib
- J2, J3, J4, J5: symbol Arduino_uno_sheild-rescue:6posheader-JPL_Robotics_Lib -> Arduino_uno_shield-rescue:6posheader-JPL_Robotics_Lib
- J6: symbol Arduino_uno_sheild-rescue:ED2580-ND-JPL_Robotics_Lib -> Arduino_uno_shield-rescue:ED2580-ND-JPL_Robotics_Lib
- y1: symbol Arduino_uno_sheild-rescue:rover_silkscreen -> Arduino_uno_shield-rescue:rover_silkscreen
Changed lines of the file:
@@
 $EndComp
 $Comp
-L Arduino_uno_sheild-rescue:6posheader-JPL_Robotics_Lib J5
+L Arduino_uno_shield-rescue:6posheader-JPL_Robotics_Lib J5
 U 1 1 5CFE8BE4
 P 3900 3400
@@
 B2
 $Comp
-L Arduino_uno_sheild-rescue:Arduino_UNO_R3-JPL_Robotics_Lib A1
+L Arduino_uno_shield-rescue:Arduino_UNO_R3-JPL_Robotics_Lib A1
 U 1 1 5D0266BD
 P 2350 3250
 F 0 "A1" H 2975 4718 30  0000 C CNN
 F 1 "Arduino_UNO_R3" H 2975 4658 30  0000 C CNN
-F 2 "JPL Robotics:Arduino Uno Sheild" H 2350 3250 30  0001 C CNN
+F 2 "JPL Robotics:Arduino Uno Shield" H 2350 3250 30  0001 C CNN
 F 3 "" H 2350 3250 30  0001 C CNN
 	1    2350 3250
@@
 CLK
 $Comp
-L Arduino_uno_sheild-rescue:ED2580-ND-JPL_Robotics_Lib J6
+L Arduino_uno_shield-rescue:ED2580-ND-JPL_Robotics_Lib J6
 U 1 1 5D02F3BE
 P 4900 3300
@@
 	5200 3250 5200 3350
 $Comp
-L Arduino_uno_sheild-rescue:ED10523-ND-JPL_Robotics_Lib J1
+L Arduino_uno_shield-rescue:ED10523-ND-JPL_Robotics_Lib J1
 U 1 1 5D03196E
 P 2550 3750
@@
 GND
 $Comp
-L Arduino_uno_sheild-rescue:6posheader-JPL_Robotics_Lib J2
+L Arduino_uno_shield-rescue:6posheader-JPL_Robotics_Lib J2
 U 1 1 5D037B9E
 P 3900 1800
@@
 	4100 1750 4200 1750
 $Comp
-L Arduino_uno_sheild-rescue:6posheader-JPL_Robotics_Lib J3
+L Arduino_uno_shield-rescue:6posheader-JPL_Robotics_Lib J3
 U 1 1 5D04118C
 P 3900 2200
@@
 	4100 2150 4200 2150
 $Comp
-L Arduino_uno_sheild-rescue:6posheader-JPL_Robotics_Lib J4
+L Arduino_uno_shield-rescue:6posheader-JPL_Robotics_Lib J4
 U 1 1 5D0426DF
 P 3900 2600
@@
 Connection ~ 4400 3150
 $Comp
-L Arduino_uno_sheild-rescue:rover_silkscreen y1
+L Arduino_uno_shield-rescue:rover_silkscreen y1
 U 1 1 5D3EF344
 P 2500 4050
